File: schematic/color_access_granter.sch (EAGLE design)
At the start: 14 parts, among them IC2 MEGA324-P, U1 HC_05

Commit message: Modified electronic schematic
Changed lines of the file:
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@@
 <part name="GND1" library="supply1" library_urn="urn:adsk.eagle:library:371" deviceset="GND" device=""/>
 <part name="GND2" library="supply1" library_urn="urn:adsk.eagle:library:371" deviceset="GND" device=""/>
-<part name="C1" library="docu-dummy" library_urn="urn:adsk.eagle:library:215" deviceset="C" device=""/>
 <part name="VDD1" library="supply1" library_urn="urn:adsk.eagle:library:371" deviceset="VDD" device=""/>
 <part name="U1" library="Bluetooth HC-05" deviceset="HC_05" device=""/>
@@
 <instance part="GND1" gate="1" x="144.722478125" y="43.737821875" rot="R180"/>
 <instance part="GND2" gate="1" x="228.6" y="119.38" rot="R90"/>
-<instance part="C1" gate="G$1" x="218.44" y="109.22" rot="R90"/>
 <instance part="VDD1" gate="G$1" x="231.14" y="109.22" rot="R270"/>
 <instance part="U1" gate="G$1" x="220.98" y="45.72"/>
@@
 </segment>
 </net>
-<net name="N$2" class="0">
-<segment>
+<net name="VDD" class="0">
+<segment>
+<pinref part="VDD1" gate="G$1" pin="VDD"/>
 <portref moduleinst="TCS230-1" port="VDD"/>
-<wire x1="200.66" y1="109.22" x2="215.9" y2="109.22" width="0.1524" layer="91"/>
-</segment>
-</net>
-<net name="VDD" class="0">
-<segment>
-<pinref part="VDD1" gate="G$1" pin="VDD"/>
-<wire x1="223.52" y1="109.22" x2="228.6" y2="109.22" width="0.1524" layer="91"/>
-</segment>
-</net>
+<wire x1="200.66" y1="109.22" x2="228.6" y2="109.22" width="0.1524" layer="91"/>
+</segment>
+</net>
